File: Bus-proto/Universal-proto-v1.kicad_pcb (KiCad board)
At the start: 2 copper layers, 81.5 x 121 mm, 52 parts, among them J1 Bus_ISA_8bit, J2 ISA Breakout, J3 Pico GPIO Breakout 2, J4 Pico GPIO Breakout 1, J5 Conn_01x20, J6 Conn_01x20, J7 Conn_01x20, J8 Conn_01x20, J9 Conn_02x02_Odd_Even

Commit message: M3 mounting holes with ground connection
Parts:
- added REF**: MountingHole_3.2mm_M3_DIN965_Pad_TopBottom, MountingHole:MountingHole_3.2mm_M3_DIN965_Pad_TopBottom, F.Cu at (110.7, 26.4)
- added REF**: MountingHole_3.2mm_M3_DIN965_Pad_TopBottom, MountingHole:MountingHole_3.2mm_M3_DIN965_Pad_TopBottom, F.Cu at (184.9, 26.4)
Routing:
- net /GND: track 340.4 -> 438.8 mm

Commit message: Update version date
Other:
- board text added: "v2026-APR-2"
- board text removed: "v2026-MAR-27"
Changed lines of the file:
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@@
 			(at 0 3.75 0)
 			(layer "F.Fab")
+			(hide yes)
 			(effects
 				(font
@@
 			(at 0 3.75 0)
 			(layer "F.Fab")
+			(hide yes)
 			(effects
 				(font
@@
 		)
 	)
-	(gr_text "v2026-MAR-27"
-		(at 174.45 130.81 -0)
+	(gr_text "v2026-APR-2"
+		(at 174.45 130.81 0)
 		(layer "F.SilkS")
 		(effects

Commit message: Fix edge cuts and labels
Other:
- board size 81.5 x 121 mm -> 81.5 x 112 mm
- board text added: "v2026-APR-19"
- board text removed: "v2026-APR-2"

Commit message: Fix edges
Other:
- board size 81.5 x 112 mm -> 81.3 x 112 mm
Changed lines of the file:
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@@
 		(attr exclude_from_pos_files)
 		(fp_line
-			(start -78.24 2.54)
-			(end -78.24 -5)
+			(start -78.74 2.54)
+			(end -78.74 -5)
 			(stroke
 				(width 0.1)
@@
 		)
 		(fp_line
-			(start 0.77 3.81)
-			(end -76.97 3.81)
+			(start 1.27 3.81)
+			(end -77.47 3.81)
 			(stroke
 				(width 0.1)
@@
 		)
 		(fp_line
-			(start 2.04 -5.08)
-			(end 2.04 2.54)
+			(start 2.54 -5.08)
+			(end 2.54 2.54)
 			(stroke
 				(width 0.1)
@@
 		)
 		(fp_arc
-			(start -76.97 3.81)
-			(mid -77.868026 3.438026)
-			(end -78.24 2.54)
+			(start -77.47 3.81)
+			(mid -78.368026 3.438026)
+			(end -78.74 2.54)
 			(stroke
 				(width 0.1)
@@
 		)
 		(fp_arc
-			(start 2.04 2.54)
-			(mid 1.668026 3.438026)
-			(end 0.77 3.81)
+			(start 2.54 2.54)
+			(mid 2.168026 3.438026)
+			(end 1.27 3.81)
 			(stroke
 				(width 0.1)
@@
 	)
 	(gr_line
-		(start 107 22.966)
-		(end 188.5 22.966)
+		(start 107.12 22.966)
+		(end 188.4 22.966)
 		(stroke
 			(width 0.127)
@@
 	)
 	(gr_line
-		(start 188.5 22.966)
-		(end 188.5 134.92)
+		(start 188.4 22.966)
+		(end 188.4 134.92)
 		(stroke
 			(width 0.127)
@@
 	)
 	(gr_line
-		(start 107 22.966)
-		(end 107 135)
-		(stroke
-			(width 0.127)
-			(type default)
-		)
-		(layer "Edge.Cuts")
-	)
-	(gr_line
-		(start 107.62 135)
-		(end 107 135)
-		(stroke
-			(width 0.127)
-			(type default)
-		)
-		(layer "Edge.Cuts")
-	)
-	(gr_line
-		(start 187.9 134.92)
-		(end 188.5 134.92)
+		(start 107.12 22.966)
+		(end 107.12 135)
 		(stroke
 			(width 0.127)
