File: Bus-proto/Universal-proto-v1.kicad_pcb (KiCad board)
At the start: 2 copper layers, 81.3 x 112 mm, 54 parts, among them J1 Bus_ISA_8bit, J2 ISA Breakout, J3 Pico GPIO Breakout 2, J4 Pico GPIO Breakout 1, J5 Conn_01x20, J6 Conn_01x20, J7 Conn_01x20, J8 Conn_01x20, J9 Conn_02x02_Odd_Even

Commit message: Fix GPIO label
Other:
- board text removed: "GP5_ISA_D5"
Changed lines of the file:
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@@
 		)
 	)
-	(gr_text "GP5_ISA_D5"
+	(gr_text "GP25_ISA_D5"
 		(at 178.74 106.35 90)
 		(layer "F.SilkS")
